Commit message: Switch to Model T42 gripper

File: src/Universal_Robots_ROS2_Description/urdf/gripper.urdf.xacro (robot description, xacro)
@@ -1,317 +1,300 @@
 <?xml version="1.0"?>
-<robot xmlns:xacro="http://wiki.ros.org/xacro" name="robotiq_2f_85_gripper">
-  <xacro:macro name="robotiq_85_gripper" params="tf_prefix">
-    <xacro:macro name = "material_color">
-      <material name = "black">
-        <color rgba = "0.7 0.7 0.7 1"/>
-      </material>
-    </xacro:macro>
-    <link name="robotiq_85_base_link">
-      <inertial>
-        <origin xyz="0.00021987 -2.3546E-10 0.030163" rpy="0 0 0"/>
-        <mass value="0.30915" />
-        <inertia ixx="0.00028972" ixy="-5.7879E-10" ixz="-1.8543E-06" iyy="0.00030737" iyz="1.682E-12" izz="0.00019914" />
-      </inertial>
-      <visual>
-        <origin xyz="0 0 0" rpy="0 0 0" />
-        <geometry>
-          <mesh filename="model://ur_description/meshes/robotiq_gripper/robotiq_85_base_link_fine.STL" />
-        </geometry>
-        <xacro:material_color/>
-      </visual>
-      <collision>
-        <origin xyz="0 0 0" rpy="0 0 0" />
-        <geometry>
-          <mesh filename="model://ur_description/meshes/robotiq_gripper/robotiq_85_base_link_coarse.STL" />
-        </geometry>
-      </collision>
-    </link>
-    <joint name="${tf_prefix}flange_robotiq_85_base_link" type="fixed">
+<robot xmlns:xacro="http://wiki.ros.org/xacro" name="t42">
+  <xacro:macro name="t42_gripper" params="tf_prefix">
+    <link name="hand_base" />
+    <joint name="${tf_prefix}flange_hand_base" type="fixed">
         <parent link="${tf_prefix}flange" />
-        <child link="robotiq_85_base_link" />
-        <origin xyz="0 0 0" rpy="0 1.57 0" />
-      </joint>
-    <link name="left_outer_knuckle">
-      <inertial>
-        <origin xyz="0.0178331863169983 3.68915177224286E-11 0.0021442477325704" rpy="0 0 0" />
-        <mass value="0.00684838849434396" />
-        <inertia ixx="2.66832029033166E-07" ixy="1.66142314639824E-15" ixz="1.45945633322873E-07"
-               iyy="1.3889233257419E-06" iyz="2.82951161241588E-15" izz="1.26603336914415E-06" />
-      </inertial>
-      <visual>
-        <origin xyz="0 0 0" rpy="0 0 0" />
-        <geometry>
-          <mesh filename="model://ur_description/meshes/robotiq_gripper/outer_knuckle_fine.STL" />
-        </geometry>
-        <xacro:material_color/>
-      </visual>
-      <collision>
-        <origin xyz="0 0 0" rpy="0 0 0" />
-        <geometry>
-          <mesh filename="model://ur_description/meshes/robotiq_gripper/outer_knuckle_coarse.STL" />
-        </geometry>
-      </collision>
-    </link>
-    <joint name="finger_joint" type="revolute">
-      <origin xyz="0.0306011444260539 0 0.0627920162695395" rpy="0 0 0" />
-      <parent link="robotiq_85_base_link" />
-      <child link="left_outer_knuckle" />
-      <axis xyz="0 -1 0" />
-      <limit lower="0" upper="0.725" velocity="2.0" effort="1000" />
-    </joint>
-    <link name="left_outer_finger">
-      <inertial>
-        <origin xyz="0.00131451599174296 2.88942057994543E-15 0.0215404163180413" rpy="0 0 0" />
-        <mass value="0.0273093985570947" />
-        <inertia ixx="8.51629628283022E-06" ixy="2.58174336207405E-19" ixz="3.83829504344079E-07"
-                 iyy="6.9133328065108E-06" iyz="-7.58589926143789E-19" izz="2.25006832221981E-06" />
-      </inertial>
-      <visual>
-        <origin xyz="0 0 0" rpy="0 0 0" />
-        <geometry>
-          <mesh filename="model://ur_description/meshes/robotiq_gripper/outer_finger_fine.STL" />
-        </geometry>
-        <xacro:material_color/>
-      </visual>
-      <collision>
-        <origin xyz="0 0 0" rpy="0 0 0" />
-        <geometry>
-          <mesh filename="model://ur_description/meshes/robotiq_gripper/outer_finger_coarse.STL" />
-        </geometry>
-      </collision>
-    </link>
-    <joint name="left_outer_finger_joint" type="fixed">
-      <origin xyz="0.0316910442266543 0 -0.00193396375724605" rpy="0 0 0" />
-      <parent link="left_outer_knuckle" />
-      <child link="left_outer_finger" />
-      <axis xyz="0 -1 0" />
-    </joint>
-    <link name="left_inner_knuckle">
-      <inertial>
-        <origin xyz="0.017097546626628 -3.93808524389535E-10 0.0224918438201868" rpy="0 0 0" />
-        <mass value="0.0110930853895903" />
-        <inertia ixx="4.23392770691541E-06" ixy="5.748978936968E-15" ixz="1.78855677119788E-06"
-                 iyy="3.96548790524392E-06" iyz="1.05464666369669E-14" izz="3.24068002883007E-06" />
-      </inertial>
-      <visual>
-        <origin xyz="0 0 0" rpy="0 0 0" />
-        <geometry>
-          <mesh filename="model://ur_description/meshes/robotiq_gripper/inner_knuckle_fine.STL" />
-        </geometry>
-        <xacro:material_color/>
-      </visual>
-      <collision>
-        <origin xyz="0 0 0" rpy="0 0 0" />
-        <geometry>
-          <mesh filename="model://ur_description/meshes/robotiq_gripper/inner_knuckle_coarse.STL" />
-        </geometry>
-      </collision>
-    </link>
-    <joint name="left_inner_knuckle_joint" type="revolute">
-      <origin xyz="0.0127000000001501 0 0.0693074999999639" rpy="0 0 0" />
-      <parent link="robotiq_85_base_link" />
-      <child link="left_inner_knuckle" />
-      <axis xyz="0 -1 0" />
-      <limit lower="0" upper="0.8757" velocity="2.0" effort="1000" />
-      <mimic joint="finger_joint" multiplier="1" offset="0" />
-    </joint>
-    <link name="left_inner_finger">
-      <inertial>
-        <origin xyz="0.0060275613594574 -6.29183141465421E-15 0.00669925693133241" rpy="0 0 0" />
-        <mass value="0.00724255346165745" />
-        <inertia ixx="1.47824274053603E-06" ixy="-3.94884463570303E-19" ixz="-3.45268847648622E-07"
-                 iyy="1.70064480838395E-06" iyz="3.5059838910097E-19" izz="4.77151336838364E-07" />
-      </inertial>
-      <visual>
-        <origin xyz="0 0 0" rpy="0 0 0" />
-        <geometry>
-          <mesh filename="model://ur_description/meshes/robotiq_gripper/inner_finger_fine.STL" />
-        </geometry>
-        <xacro:material_color/>
-      </visual>
-      <collision>
-        <origin xyz="0 0 0" rpy="0 0 0" />
-        <geometry>
-          <mesh filename="model://ur_description/meshes/robotiq_gripper/inner_finger_coarse.STL" />
-        </geometry>
-      </collision>
-    </link>
-    <joint name="left_inner_finger_joint" type="revolute">
-      <origin xyz="0.034585310861294 0 0.0454970193817975" rpy="0 0 0" />
-      <parent link="left_inner_knuckle" />
-      <child link="left_inner_finger" />
-      <axis xyz="0 -1 0" />
-      <limit lower="0" upper="0.8757" velocity="2.0" effort="1000" />
-      <mimic joint="finger_joint" multiplier="-1" offset="0" />
-    </joint>
-    <link name="right_inner_knuckle">
-      <inertial>
-        <origin xyz="0.0168606186773776 3.93808471820465E-10 0.0226699950793434" rpy="0 0 0" />
-        <mass value="0.0110930853895903" />
-        <inertia ixx="4.27134775939882E-06" ixy="-8.53568456728898E-15" ixz="1.77774229944246E-06"
-                 iyy="3.96548790524392E-06" iyz="-8.45108024914164E-15" izz="3.20325997634666E-06" />
-      </inertial>
-      <visual>
-        <origin xyz="0 0 0" rpy="0 0 0" />
-        <geometry>
-          <mesh filename="model://ur_description/meshes/robotiq_gripper/inner_knuckle_fine.STL" />
-        </geometry>
-        <xacro:material_color/>
-      </visual>
-      <collision>
-        <origin xyz="0 0 0" rpy="0 0 0" />
-        <geometry>
-          <mesh filename="model://ur_description/meshes/robotiq_gripper/inner_knuckle_coarse.STL" />
-        </geometry>
-      </collision>
-    </link>
-    <joint name="right_inner_knuckle_joint" type="revolute">
-      <origin xyz="-0.0126999999998499 0 0.0693075000000361" rpy="0 0 3.14159265358979" />
-      <parent link="robotiq_85_base_link" />
-      <child link="right_inner_knuckle" />
-      <axis xyz="0 1 0" />
-      <limit lower="0" upper="0.8757" velocity="2.0" effort="1000" />
-      <mimic joint="finger_joint" multiplier="-1" offset="0" />
-    </joint>
-    <link name="right_inner_finger">
-      <inertial>
-        <origin xyz="0.00602756228812038 -6.47284509480176E-15 0.00669925609578108" rpy="0 0 0" />
-        <mass value="0.00724255346165744" />
-        <inertia ixx="1.47824283625957E-06" ixy="-3.95952064019123E-19" ixz="-3.45268708875543E-07"
-                 iyy="1.70064480838394E-06" iyz="3.55286507960029E-19" izz="4.77151241114822E-07" />
-      </inertial>
-      <visual>
-        <origin xyz="0 0 0" rpy="0 0 0" />
-        <geometry>
-          <mesh filename="model://ur_description/meshes/robotiq_gripper/inner_finger_fine.STL" />
-        </geometry>
-        <xacro:material_color/>
-      </visual>
-      <collision>
-        <origin xyz="0 0 0" rpy="0 0 0" />
-        <geometry>
-          <mesh filename="model://ur_description/meshes/robotiq_gripper/inner_finger_coarse.STL" />
-        </geometry>
-      </collision>
-    </link>
-    <joint name="right_inner_finger_joint" type="revolute">
-      <origin xyz="0.0341060475457406 0 0.0458573878541688" rpy="0 0 0" />
-      <parent link="right_inner_knuckle" />
-      <child link="right_inner_finger" />
-      <axis xyz="0 1 0" />
-      <limit lower="0" upper="0.8757" velocity="2.0" effort="1000" />
-      <mimic joint="finger_joint" multiplier="1" offset="0" />
-    </joint>
-    <link name="right_outer_knuckle">
-      <inertial>
-        <origin xyz="0.0178097074051638 3.60493211424024E-11 0.00233123458346721" rpy="0 0 0" />
-        <mass value="0.00684838849401352" />
-        <inertia ixx="2.70004361573169E-07" ixy="1.59579467624491E-15" ixz="1.56396493788199E-07"
-                 iyy="1.38892332558312E-06" iyz="2.82357800318817E-15" izz="1.26286103637978E-06" />
-      </inertial>
-      <visual>
-        <origin xyz="0 0 0" rpy="0 0 0" />
-        <geometry>
-          <mesh filename="model://ur_description/meshes/robotiq_gripper/outer_knuckle_fine.STL" />
-        </geometry>
-        <xacro:material_color/>
-      </visual>
-      <collision>
-        <origin xyz="0 0 0" rpy="0 0 0" />
-        <geometry>
-          <mesh filename="model://ur_description/meshes/robotiq_gripper/outer_knuckle_coarse.STL" />
-        </geometry>
-      </collision>
-    </link>
-    <joint name="right_outer_knuckle_joint" type="revolute">
-      <origin xyz="-0.0306011444258893 0 0.0627920162695395" rpy="0 0 3.14159265358979" />
-      <parent link="robotiq_85_base_link" />
-      <child link="right_outer_knuckle" />
-      <axis xyz="0 1 0" />
-      <limit lower="0" upper="0.8757" velocity="2.0" effort="1000" />
-      <mimic joint="finger_joint" multiplier="-1" offset="0" />
-    </joint>
-    <link name="right_outer_finger">
-      <inertial>
-        <origin xyz="0.00108844269639009 -2.611488350845E-15 0.0215530225245502" rpy="0 0 0" />
-        <mass value="0.0273093985570947" />
-        <inertia ixx="8.52366028592721E-06" ixy="3.41683380899422E-19" ixz="3.18003675694284E-07"
-                 iyy="6.91333280651081E-06" iyz="7.37726682706417E-19" izz="2.24270431912283E-06" />
-      </inertial>
-      <visual>
-        <origin xyz="0 0 0" rpy="0 0 0" />
-        <geometry>
-          <mesh filename="model://ur_description/meshes/robotiq_gripper/outer_finger_fine.STL" />
-        </geometry>
-        <xacro:material_color/>
-      </visual>
-      <collision>
-        <origin xyz="0 0 0" rpy="0 0 0" />
-        <geometry>
-          <mesh filename="model://ur_description/meshes/robotiq_gripper/outer_finger_coarse.STL" />
-        </geometry>
-      </collision>
-    </link>
-    <joint name="right_outer_finger_joint" type="fixed">
-      <origin xyz="0.0317095909367246 0 -0.0016013564954687" rpy="0 0 0" />
-      <parent link="right_outer_knuckle" />
-      <child link="right_outer_finger" />
-      <axis xyz="0 1 0" />
-    </joint>
-    <gazebo reference="left_inner_knuckle_joint">
-      <preserveFixedJoint>true</preserveFixedJoint>
-      <physics>
-        <ode>
-          <limit>
-            <cfm>0</cfm>
-            <erp>0.2</erp>
-          </limit>
-        </ode>
-      </physics>
-    </gazebo>
-    <gazebo reference="left_inner_finger_joint">
-      <preserveFixedJoint>true</preserveFixedJoint>
-      <physics>
-        <ode>
-          <limit>
-            <cfm>0</cfm>
-            <erp>0.2</erp>
-          </limit>
-        </ode>
-      </physics>
-    </gazebo>
-    <gazebo reference="right_inner_knuckle_joint">
-      <preserveFixedJoint>true</preserveFixedJoint>
-      <physics>
-        <ode>
-          <limit>
-            <cfm>0</cfm>
-            <erp>0.2</erp>
-          </limit>
-        </ode>
-      </physics>
-    </gazebo>
-    <gazebo reference="right_outer_knuckle_joint">
-      <preserveFixedJoint>true</preserveFixedJoint>
-      <physics>
-        <ode>
-          <limit>
-            <cfm>0</cfm>
-            <erp>0.2</erp>
-          </limit>
-        </ode>
-      </physics>
-    </gazebo>
-    <gazebo reference="right_inner_finger_joint">
-      <preserveFixedJoint>true</preserveFixedJoint>
-      <physics>
-        <ode>
-          <limit>
-            <cfm>0</cfm>
-            <erp>0.2</erp>
-          </limit>
-        </ode>
-      </physics>
-    </gazebo>
+        <child link="hand_base" />
+        <origin xyz="0 0 0" rpy="0 3.14 0" />
+    </joint>
+    <link name="hand_coupler">
+        <inertial>
+            <origin xyz="0.000000 0.000000 0.025400" />
+            <mass value="1.0" />
+            <inertia ixx="1000.0" ixy="0.0" ixz="0.0" iyy="1000.0" iyz="0.0" izz="1000.0" />
+        </inertial>
+        <visual>
+            <material name="lightblue">
+                <color rgba="0. 0.3 1.0 1.0" />
+            </material>
+            <origin rpy="0 1.57079632679 0" xyz="0.000000 0.000000 0.000000" />
+            <geometry>
+                <cylinder length="0.00762" radius="0.05715" />
+            </geometry>
+        </visual>
+        <collision>
+            <origin rpy="0 1.57079632679 0" xyz="0.000000 0.000000 0.000000" />
+            <geometry>
+                <cylinder length="0.00762" radius="0.05715" />
+            </geometry>
+        </collision>
+    </link>
+    <link name="motor_space">
+        <inertial>
+            <origin xyz="0.000000 0.000000 0.025400" />
+            <mass value="1.0" />
+            <inertia ixx="1000.0" ixy="0.0" ixz="0.0" iyy="1000.0" iyz="0.0" izz="1000.0" />
+        </inertial>
+        <visual>
+            <material name="black">
+                <color rgba="0. 0. 0. 1.0" />
+            </material>
+            <origin rpy="0 1.57079632679 0" xyz="0.000000 0.000000 0.000000" />
+            <geometry>
+                <cylinder length="0.0508" radius="0.04572" />
+            </geometry>
+        </visual>
+        <collision>
+            <origin rpy="0 1.57079632679 0" xyz="0.000000 0.000000 0.000000" />
+            <geometry>
+                <cylinder length="0.0508" radius="0.05715" />
+            </geometry>
+        </collision>
+    </link>
+    <link name="simple_base">
+        <inertial>
+            <origin xyz="0.000000 0.000000 0.025400" />
+            <mass value="1.0" />
+            <inertia ixx="1000.0" ixy="0.0" ixz="0.0" iyy="1000.0" iyz="0.0" izz="1000.0" />
+        </inertial>
+        <visual>
+            <material name="lightlue">
+                <color rgba="0. 0.3 1.0 1.0" />
+            </material>
+            <origin rpy="0 1.57079632679 0" xyz="0.000000 0.000000 0.000000" />
+            <geometry>
+                <cylinder length="0.00762" radius="0.05715" />
+            </geometry>
+        </visual>
+        <collision>
+            <origin rpy="0 1.57079632679 0" xyz="0.000000 0.000000 0.000000" />
+            <geometry>
+                <cylinder length="0.00762" radius="0.05715" />
+            </geometry>
+        </collision>
+    </link>
+    <link name="prox_r">
+        <inertial>
+            <origin xyz="-0.015875 -0.009000 -0.071550" />
+            <mass value="0.1" />
+            <inertia ixx="0.01" ixy="0.0" ixz="0.0" iyy="0.01" iyz="0.0" izz="0.01" />
+        </inertial>
+        <visual>
+            <material name="white">
+                <color rgba="1.0 1.0 1.0 1.0" />
+            </material>
+            <origin xyz="-0.015875 -0.009000 -0.071550" />
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
File: src/Universal_Robots_ROS2_Description/urdf/ur_macro.xacro (robot description, xacro)
@@ -364,5 +364,5 @@
     </joint>
     <xacro:include filename="$(find ur_description)/urdf/gripper.urdf.xacro" />
-    <xacro:robotiq_85_gripper tf_prefix="${tf_prefix}"/>
+    <xacro:t42_gripper tf_prefix="${tf_prefix}"/>
     <!-- ROS-Industrial 'tool0' frame - all-zeros tool frame -->
     <link name="${tf_prefix}tool0"/>
@@ -373,4 +373,6 @@
       <child link="${tf_prefix}tool0"/>
     </joint>
+    <xacro:include filename="$(find ur_description)/control/ur10e_ros2_control.urdf.xacro" />
+    <xacro:robot_arm_ros2_control name="robotname"/>
   </xacro:macro>
 </robot>
